File: LabReports/Lab4/controller_board.brd (EAGLE design)
At the start: 185 x 33 mm, 12 parts, among them J1 JST_3PIN_GND_VDD_SIG, J2 JST_3PIN_GND_VDD_SIG, J3 JST_3PIN_GND_VDD_SIG, J4 JST_3PIN_GND_VDD_SIG, J5 GIMBAL_3PIN_MATCH_TDOCU

Commit message: Added resistors to schematic, but can't route with free version
Parts:
- added R1, R2, R3, R4: 3.3K, Trevor-lab4:CFR-12
Connections:
- new net N$1: J1.2, R1.P$1
- new net N$2: J2.2, R2.P$1
- new net N$3: J3.2, R3.P$1
- new net N$4: J4.2, R4.P$1
- net 3.3V: now also R1.P$2, R2.P$2, R3.P$2, R4.P$2; no longer J1.2, J2.2, J3.2, J4.2
Changed lines of the file:
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@@
 <layer number="17" name="Pads" color="2" fill="1" visible="yes" active="yes"/>
 <layer number="18" name="Vias" color="2" fill="1" visible="yes" active="yes"/>
-<layer number="19" name="Unrouted" color="6" fill="1" visible="no" active="yes"/>
+<layer number="19" name="Unrouted" color="6" fill="1" visible="yes" active="yes"/>
 <layer number="20" name="Dimension" color="15" fill="1" visible="yes" active="yes"/>
 <layer number="21" name="tPlace" color="7" fill="1" visible="yes" active="yes"/>
@@
 <element name="U$1" library="Controller" package="CONNECTOR_BOARD_OUTLINE" value="" x="0" y="0"/>
 <element name="U$2" library="Controller" package="BUTTON-TACTILE-SQUARE-ADAFRUIT1010" value="BUTTON-TACTILE-SQUARE" x="152.719" y="31.166" locked="yes" rot="R180"/>
+<element name="R1" library="Trevor-lab4" package="CFR-12" value="3.3K" x="92.143" y="37.057">
+<attribute name="CREATOR" value="Trevor Smith" x="92.143" y="37.057" size="1.778" layer="27" display="off"/>
+<attribute name="DISTPN" value="*EBK-ND" x="92.143" y="37.057" size="1.778" layer="27" display="off"/>
+<attribute name="DIST" value="Digikey" x="92.143" y="37.057" size="1.778" layer="27" display="off"/>
+<attribute name="TOL" value="5%" x="92.143" y="37.057" size="1.778" layer="27" display="off"/>
+</element>
+<element name="R2" library="Trevor-lab4" package="CFR-12" value="3.3K" x="89.113" y="26.793">
+<attribute name="CREATOR" value="Trevor Smith" x="89.113" y="26.793" size="1.778" layer="27" display="off"/>
+<attribute name="DISTPN" value="*EBK-ND" x="89.113" y="26.793" size="1.778" layer="27" display="off"/>
+<attribute name="DIST" value="Digikey" x="89.113" y="26.793" size="1.778" layer="27" display="off"/>
+<attribute name="TOL" value="5%" x="89.113" y="26.793" size="1.778" layer="27" display="off"/>
+</element>
+<element name="R3" library="Trevor-lab4" package="CFR-12" value="3.3K" x="70.866" y="37.49">
+<attribute name="CREATOR" value="Trevor Smith" x="70.866" y="37.49" size="1.778" layer="27" display="off"/>
+<attribute name="DISTPN" value="*EBK-ND" x="70.866" y="37.49" size="1.778" layer="27" display="off"/>
+<attribute name="DIST" value="Digikey" x="70.866" y="37.49" size="1.778" layer="27" display="off"/>
+<attribute name="TOL" value="5%" x="70.866" y="37.49" size="1.778" layer="27" display="off"/>
+</element>
+<element name="R4" library="Trevor-lab4" package="CFR-12" value="3.3K" x="80.772" y="37.555">
+<attribute name="CREATOR" value="Trevor Smith" x="80.772" y="37.555" size="1.778" layer="27" display="off"/>
+<attribute name="DISTPN" value="*EBK-ND" x="80.772" y="37.555" size="1.778" layer="27" display="off"/>
+<attribute name="DIST" value="Digikey" x="80.772" y="37.555" size="1.778" layer="27" display="off"/>
+<attribute name="TOL" value="5%" x="80.772" y="37.555" size="1.778" layer="27" display="off"/>
+</element>
 </elements>
 <signals>
 <signal name="3.3V">
-<contactref element="J1" pad="2"/>
-<contactref element="J2" pad="2"/>
-<contactref element="J3" pad="2"/>
-<contactref element="J4" pad="2"/>
 <contactref element="J5" pad="1"/>
 <contactref element="JP1" pad="2"/>
 <contactref element="U$2" pad="P2"/>
 <contactref element="U$2" pad="P"/>
+<contactref element="R1" pad="P$2"/>
+<contactref element="R2" pad="P$2"/>
+<contactref element="R3" pad="P$2"/>
+<contactref element="R4" pad="P$2"/>
+<wire x1="146.719" y1="28.666" x2="158.719" y2="28.666" width="0" layer="19" extent="1-1"/>
+<wire x1="133" y1="25" x2="146.719" y2="28.666" width="0" layer="19" extent="1-1"/>
 <wire x1="105" y1="49.46" x2="133" y2="25" width="0" layer="19" extent="1-1"/>
-<wire x1="133" y1="25" x2="146.719" y2="28.666" width="0" layer="19" extent="1-1"/>
-<wire x1="146.719" y1="28.666" x2="158.719" y2="28.666" width="0" layer="19" extent="1-1"/>
-<wire x1="158.719" y1="28.666" x2="186" y2="51" width="0" layer="19" extent="1-1"/>
-<wire x1="200" y1="28" x2="186" y2="51" width="0" layer="19" extent="1-1"/>
-<wire x1="71" y1="49" x2="83" y2="49" width="0" layer="19" extent="1-1"/>
-<wire x1="83" y1="49" x2="105" y2="49.46" width="0" layer="19" extent="1-1"/>
+<wire x1="95.143" y1="37.057" x2="105" y2="49.46" width="0" layer="19" extent="1-1"/>
+<wire x1="92.113" y1="26.793" x2="95.143" y2="37.057" width="0" layer="19" extent="1-1"/>
+<wire x1="73.866" y1="37.49" x2="92.113" y2="26.793" width="0" layer="19" extent="1-1"/>
+<wire x1="83.772" y1="37.555" x2="73.866" y2="37.49" width="0" layer="19" extent="1-1"/>
 </signal>
 <signal name="GND">
@@
 <wire x1="83" y1="47" x2="126" y2="52.62" width="0" layer="19" extent="1-1"/>
 </signal>
+<signal name="N$1">
+<contactref element="J1" pad="2"/>
+<contactref element="R1" pad="P$1"/>
+<wire x1="89.143" y1="37.057" x2="186" y2="51" width="0" layer="19" extent="1-1"/>
+</signal>
+<signal name="N$2">
+<contactref element="J2" pad="2"/>
+<contactref element="R2" pad="P$1"/>
+<wire x1="86.113" y1="26.793" x2="200" y2="28" width="0" layer="19" extent="1-1"/>
+</signal>
+<signal name="N$3">
+<contactref element="J3" pad="2"/>
+<contactref element="R3" pad="P$1"/>
+<wire x1="67.866" y1="37.49" x2="71" y2="49" width="0" layer="19" extent="1-1"/>
+</signal>
+<signal name="N$4">
+<contactref element="J4" pad="2"/>
+<contactref element="R4" pad="P$1"/>
+<wire x1="77.772" y1="37.555" x2="83" y2="49" width="0" layer="19" extent="1-1"/>
+</signal>
 </signals>

Commit message: Routed board and processed CAM
Parts:
- moved R2 108.0 mm to (197.0, 31.9), turned to 180 degrees
- moved R1 86.6 mm to (178.0, 48.0), turned to 270 degrees
- moved R3 13.3 mm to (83.0, 43.0)
- moved R4 13.3 mm to (91.0, 46.0), turned to 270 degrees
Routing:
- net GND: track 0.00 -> 190.8 mm
- net 3.3V: track 0.00 -> 134.5 mm
- net ROLL: track 0.00 -> 80.1 mm, vias 0 -> 2
- net THROTTLE: track 0.00 -> 66.0 mm
- net PITCH: track 0.00 -> 64.1 mm
- net N$9: track 0.00 -> 53.1 mm
- net YAW: track 0.00 -> 47.8 mm, vias 0 -> 2
- net N$6: track 0.00 -> 37.4 mm
- net N$3: track 0.00 -> 11.5 mm
- net N$4: track 0.00 -> 8.00 mm
- net N$1: track 0.00 -> 8.00 mm
- net N$2: track 0.00 -> 3.90 mm
Other:
- board text added: "CSE 190 Spring 2015"
- board text added: "Controller Board r1"
- board text added: "Trevor Smith"
