File: LabReports/Lab4/controller_board.sch (EAGLE design)
At the start: 11 parts, among them J1 JST_3PIN_GND_VDD_SIG, J2 JST_3PIN_GND_VDD_SIG, J3 JST_3PIN_GND_VDD_SIG, J4 JST_3PIN_GND_VDD_SIG, J5 GIMBAL_3PIN_MATCH_TDOCU

Commit message: Added resistors to schematic, but can't route with free version
Parts:
- added R1, R2, R3, R4: 3.3K, Trevor-lab4:RESISTOR-CFR12
Connections:
- new net N$1: J1.VDD, R1.P$1
- new net N$2: J2.VDD, R2.P$1
- new net N$3: J3.VDD, R3.P$1
- new net N$4: J4.VDD, R4.P$1
- net 3.3V: now also R1.P$2, R2.P$2, R3.P$2, R4.P$2; no longer J1.VDD, J2.VDD, J3.VDD, J4.VDD
