File: LabReports/Lab5/quadcopter-smith.brd (EAGLE design)
At the start: 95.4 x 95.4 mm, 58 parts, among them J1 AVR_SPI_PRG_6NS, Q1 SI2302CDS, Q2 SI2302CDS, Q3 SI2302CDS, Q4 SI2302CDS, U1 ATMEGA128RFA1, U2 LSM9DS0-LGA24, Y1 16MHz

Commit message: for reals this time
Other:
- board size 95.4 x 95.4 mm -> 101.5 x 101.5 mm
- board text removed: "DEBUGGER"
- board text removed: "GND"
- board text removed: "X"
- board text removed: "Y"
Changed lines of the file:
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@@
 <board>
 <plain>
-<circle x="43.5" y="43.5" radius="4.2" width="0.4064" layer="20"/>
-<circle x="43.5" y="-43.5" radius="4.2" width="0.4064" layer="20"/>
-<circle x="-43.5" y="-43.5" radius="4.2" width="0.4064" layer="20"/>
-<circle x="-43.5" y="43.5" radius="4.2" width="0.4064" layer="20"/>
 <wire x1="-22.5" y1="19.5" x2="-22.5" y2="-19.5" width="0.4064" layer="20"/>
-<wire x1="-22.5" y1="-19.5" x2="-42.5" y2="-39.5" width="0.4064" layer="20"/>
-<wire x1="-42.5" y1="-39.5" x2="-39.5" y2="-42.5" width="0.4064" layer="20"/>
-<wire x1="-39.5" y1="-42.5" x2="-19.5" y2="-22.5" width="0.4064" layer="20"/>
 <wire x1="-19.5" y1="-22.5" x2="19.5" y2="-22.5" width="0.4064" layer="20"/>
-<wire x1="19.5" y1="-22.5" x2="39.5" y2="-42.5" width="0.4064" layer="20"/>
-<wire x1="39.5" y1="-42.5" x2="42.5" y2="-39.5" width="0.4064" layer="20"/>
-<wire x1="42.5" y1="-39.5" x2="22.5" y2="-19.5" width="0.4064" layer="20"/>
 <wire x1="22.5" y1="-19.5" x2="22.5" y2="19.5" width="0.4064" layer="20"/>
-<wire x1="22.5" y1="19.5" x2="42.5" y2="39.5" width="0.4064" layer="20"/>
-<wire x1="42.5" y1="39.5" x2="39.5" y2="42.5" width="0.4064" layer="20"/>
-<wire x1="39.5" y1="42.5" x2="19.5" y2="22.5" width="0.4064" layer="20"/>
 <wire x1="19.5" y1="22.5" x2="-19.5" y2="22.5" width="0.4064" layer="20"/>
-<wire x1="-19.5" y1="22.5" x2="-39.5" y2="42.5" width="0.4064" layer="20"/>
-<wire x1="-39.5" y1="42.5" x2="-42.5" y2="39.5" width="0.4064" layer="20"/>
-<wire x1="-42.5" y1="39.5" x2="-22.5" y2="19.5" width="0.4064" layer="20"/>
-<text x="17.5" y="-3.25" size="1" layer="21" ratio="10">GND</text>
-<text x="-17" y="-2.75" size="1" layer="21" ratio="10" rot="R270">DEBUGGER</text>
-<text x="-20.25" y="1.75" size="1" layer="21" ratio="10">GND</text>
-<wire x1="16.5" y1="-2.75" x2="17.25" y2="-2.75" width="0.2" layer="21"/>
-<wire x1="19" y1="-1.5" x2="19" y2="-2" width="0.2" layer="21"/>
-<wire x1="-19" y1="1" x2="-19" y2="1.5" width="0.2" layer="21"/>
-<wire x1="1" y1="-2.75" x2="-0.25" y2="-2.75" width="0.2" layer="25"/>
-<wire x1="-0.25" y1="-2.75" x2="-0.5" y2="-2.5" width="0.2" layer="25"/>
-<wire x1="-3.75" y1="-14.5" x2="-3.75" y2="-13.25" width="0.1" layer="21"/>
-<wire x1="-3.75" y1="-13.25" x2="-4" y2="-13.75" width="0.1" layer="21"/>
-<wire x1="-3.75" y1="-13.25" x2="-3.5" y2="-13.75" width="0.1" layer="21"/>
-<wire x1="-3.75" y1="-14.5" x2="-5" y2="-14.5" width="0.1" layer="21"/>
-<wire x1="-5" y1="-14.5" x2="-4.5" y2="-14.25" width="0.1" layer="21"/>
-<wire x1="-5" y1="-14.5" x2="-4.5" y2="-14.75" width="0.1" layer="21"/>
-<text x="-4.25" y="-13" size="1" layer="21">X</text>
-<text x="-5.75" y="-14.75" size="1" layer="21">Y</text>
+<wire x1="-19.5" y1="22.5" x2="-36.5" y2="39.5" width="0.4064" layer="20"/>
+<wire x1="-39.5" y1="36.5" x2="-22.5" y2="19.5" width="0.4064" layer="20"/>
+<wire x1="-39.5" y1="36.5" x2="-49.75" y2="46.75" width="0.4064" layer="20" curve="-150"/>
+<wire x1="-36.5" y1="39.5" x2="-46.75" y2="49.75" width="0.4064" layer="20" curve="150"/>
+<wire x1="-47.25" y1="45.5" x2="-45.5" y2="47.25" width="0.4064" layer="20" curve="325.75"/>
+<wire x1="-47.25" y1="45.5" x2="-49.75" y2="46.75" width="0.4064" layer="20"/>
+<wire x1="-45.5" y1="47.25" x2="-46.75" y2="49.75" width="0.4064" layer="20"/>
+<wire x1="22.5" y1="19.5" x2="39.5" y2="36.5" width="0.4064" layer="20"/>
+<wire x1="36.5" y1="39.5" x2="19.5" y2="22.5" width="0.4064" layer="20"/>
+<wire x1="36.5" y1="39.5" x2="46.75" y2="49.75" width="0.4064" layer="20" curve="-150"/>
+<wire x1="39.5" y1="36.5" x2="49.75" y2="46.75" width="0.4064" layer="20" curve="150"/>
+<wire x1="45.5" y1="47.25" x2="47.25" y2="45.5" width="0.4064" layer="20" curve="325.75"/>
+<wire x1="45.5" y1="47.25" x2="46.75" y2="49.75" width="0.4064" layer="20"/>
+<wire x1="47.25" y1="45.5" x2="49.75" y2="46.75" width="0.4064" layer="20"/>
+<wire x1="-22.5" y1="-19.5" x2="-39.5" y2="-36.5" width="0.4064" layer="20"/>
+<wire x1="-36.5" y1="-39.5" x2="-19.5" y2="-22.5" width="0.4064" layer="20"/>
+<wire x1="-36.5" y1="-39.5" x2="-46.75" y2="-49.75" width="0.4064" layer="20" curve="-150"/>
+<wire x1="-39.5" y1="-36.5" x2="-49.75" y2="-46.75" width="0.4064" layer="20" curve="150"/>
+<wire x1="-45.5" y1="-47.25" x2="-47.25" y2="-45.5" width="0.4064" layer="20" curve="325.75"/>
+<wire x1="-45.5" y1="-47.25" x2="-46.75" y2="-49.75" width="0.4064" layer="20"/>
+<wire x1="-47.25" y1="-45.5" x2="-49.75" y2="-46.75" width="0.4064" layer="20"/>
+<wire x1="19.5" y1="-22.5" x2="36.5" y2="-39.5" width="0.4064" layer="20"/>
+<wire x1="39.5" y1="-36.5" x2="22.5" y2="-19.5" width="0.4064" layer="20"/>
+<wire x1="39.5" y1="-36.5" x2="49.75" y2="-46.75" width="0.4064" layer="20" curve="-150"/>
+<wire x1="36.5" y1="-39.5" x2="46.75" y2="-49.75" width="0.4064" layer="20" curve="150"/>
+<wire x1="47.25" y1="-45.5" x2="45.5" y2="-47.25" width="0.4064" layer="20" curve="325.75"/>
+<wire x1="47.25" y1="-45.5" x2="49.75" y2="-46.75" width="0.4064" layer="20"/>
+<wire x1="45.5" y1="-47.25" x2="46.75" y2="-49.75" width="0.4064" layer="20"/>
 </plain>
 <attributes>
@@
 </class>
 </classes>
-<designrules name="default">
+<designrules name="4pcb-33board">
 <description language="de">&lt;b&gt;EAGLE Design Rules&lt;/b&gt;
 &lt;p&gt;
-Die Standard-Design-Rules sind so gewÃ¤hlt, dass sie fÃ¼r
+Die Standard-Design-Rules sind so gewählt, dass sie für
 die meisten Anwendungen passen. Sollte ihre Platine
 besondere Anforderungen haben, treffen Sie die erforderlichen
@@
 design rules under a new name.</description>
 <param name="layerSetup" value="(1*16)"/>
-<param name="mtCopper" value="0.035mm 0.035mm 0.035mm 0.035mm 0.035mm 0.035mm 0.035mm 0.035mm 0.035mm 0.035mm 0.035mm 0.035mm 0.035mm 0.035mm 0.035mm 0.035mm"/>
-<param name="mtIsolate" value="1.5mm 0.15mm 0.2mm 0.15mm 0.2mm 0.15mm 0.2mm 0.15mm 0.2mm 0.15mm 0.2mm 0.15mm 0.2mm 0.15mm 0.2mm"/>
-<param name="mdWireWire" value="8mil"/>
-<param name="mdWirePad" value="8mil"/>
-<param name="mdWireVia" value="8mil"/>
-<param name="mdPadPad" value="8mil"/>
-<param name="mdPadVia" value="8mil"/>
-<param name="mdViaVia" value="8mil"/>
-<param name="mdSmdPad" value="8mil"/>
-<param name="mdSmdVia" value="8mil"/>
-<param name="mdSmdSmd" value="8mil"/>
+<param name="mtCopper" value="0.035559375mm 0.035559375mm 0.035559375mm 0.035559375mm 0.035559375mm 0.035559375mm 0.035559375mm 0.035559375mm 0.035559375mm 0.035559375mm 0.035559375mm 0.035559375mm 0.035559375mm 0.035559375mm 0.035559375mm 0.035559375mm"/>
+<param name="mtIsolate" value="1.501140625mm 0.149859375mm 0.200659375mm 0.149859375mm 0.200659375mm 0.149859375mm 0.200659375mm 0.149859375mm 0.200659375mm 0.149859375mm 0.200659375mm 0.149859375mm 0.200659375mm 0.149859375mm 0.200659375mm"/>
+<param name="mdWireWire" value="6mil"/>
+<param name="mdWirePad" value="6mil"/>
+<param name="mdWireVia" value="6mil"/>
+<param name="mdPadPad" value="6mil"/>
+<param name="mdPadVia" value="6mil"/>
+<param name="mdViaVia" value="6mil"/>
+<param name="mdSmdPad" value="6mil"/>
+<param name="mdSmdVia" value="6mil"/>
+<param name="mdSmdSmd" value="6mil"/>
 <param name="mdViaViaSameLayer" value="8mil"/>
 <param name="mnLayersViaInSmd" value="2"/>
-<param name="mdCopperDimension" value="40mil"/>
-<param name="mdDrill" value="8mil"/>
+<param name="mdCopperDimension" value="10mil"/>
+<param name="mdDrill" value="10mil"/>
 <param name="mdSmdStop" value="0mil"/>
-<param name="msWidth" value="10mil"/>
-<param name="msDrill" value="24mil"/>
-<param name="msMicroVia" value="9.99mm"/>
+<param name="msWidth" value="6mil"/>
+<param name="msDrill" value="15mil"/>
+<param name="msMicroVia" value="9.98981875mm"/>
 <param name="msBlindViaRatio" value="0.5"/>
 <param name="rvPadTop" value="0.25"/>
